Commit message: 132

File: install/ayuda_description/share/ayuda_description/urdf/camera.xacro (robot description, xacro)
@@ -2,5 +2,5 @@
 <robot xmlns:xacro="http://www.ros.org/wiki/xacro" >
     <joint name="camera_joint" type="fixed">
-        <parent link="chassis"/>
+        <parent link="base_plate"/>
         <child link="camera_link"/>
         <origin xyz="0.276 0 0.181" rpy="0 0.18 0"/>

File: install/ayuda_description/share/ayuda_description/urdf/lidar.xacro (robot description, xacro)
@@ -2,21 +2,25 @@
 <robot xmlns:xacro="http://www.ros.org/wiki/xacro" >
     <joint name="laser_joint" type="fixed">
-        <parent link="chassis"/>
+        <parent link="front_beam"/>
         <child link="laser_frame"/>
-        <origin xyz="0.122 0 0.212" rpy="0 0 0"/>
+        <origin xyz="0.02 0 0.095" rpy="0 0 0"/>
     </joint>
     <link name="laser_frame">
         <visual>
             <geometry>
-                <cylinder radius="0.05" length="0.04"/>
+                <cylinder radius="0.03" length="0.03"/>
             </geometry>
-            <material name="black"/>
+            <material name="black">
+                <color rgba="0 0 0 1"/>
+            </material>
         </visual>
         <visual>
-            <origin xyz="0 0 -0.05"/>
+            <origin xyz="0 0 -0.03"/>
             <geometry>
-                <cylinder radius="0.01" length="0.1"/>
+                <cylinder radius="0.04" length="0.035"/>
             </geometry>
-            <material name="black"/>
+            <material name="red">
+                <color rgba="1 0 0 1"/>
+            </material>
         </visual>
         <collision>
@@ -25,10 +29,10 @@
             </geometry>
         </collision>
-        <xacro:inertial_cylinder mass="0.1" length="0.04" radius="0.05">
+        <xacro:inertial_cylinder mass="0.1" length="0.03" radius="0.03">
             <origin xyz="0 0 0" rpy="0 0 0"/>
         </xacro:inertial_cylinder>
     </link>
     <gazebo reference="laser_frame">
-        <material>Gazebo/Black</material>
+        <material>Gazebo/Red</material>
         <sensor name="laser" type="ray">
             <pose> 0 0 0 0 0 0 </pose>

File: install/ayuda_description/share/ayuda_description/urdf/n_robot_core.xacro (robot description, xacro)
@@ -26,12 +26,12 @@
     <!-- CHASSIS LINK -->
     <joint name="base_joint" type="fixed">
-        <parent link="base_footprint"/>
+        <parent link="base_link"/>
         <child link="base_plate"/>
-        <origin xyz="${-wheel_offset_x/2} 0 ${wheel_offset_z}"/>
+        <origin xyz="${-(wheel_offset_x)/2-0.04} 0 ${wheel_offset_z}"/>
     </joint>
     <link name="base_plate">
         <visual>
             <geometry>
-                <box size="0.38 .28 .05" />
+                <box size="0.34 .28 .05" />
             </geometry>
             <origin rpy="0 0 0" xyz="0 0 0.025" />
@@ -43,11 +43,39 @@
             <origin xyz="0 0 .025"/>
             <geometry>
-                <box size="0.38 0.28 0.05"/>
-            </geometry>
-        </collision>
-        <xacro:inertial_box mass="0.5" x="0.38" y="0.28" z="0.05">
+                <box size="0.34 0.28 0.05"/>
+            </geometry>
+        </collision>
+        <xacro:inertial_box mass="0.5" x="0.34" y="0.28" z="0.05">
             <origin xyz="0 0 0" rpy="0 0 0"/>
         </xacro:inertial_box>
     </link>
+    <joint name="front_beam_joint" type="fixed">
+        <parent link="base_plate"/>
+        <child link="front_beam"/>
+        <origin xyz="${wheel_offset_x/2+0.04} 0 ${-0.025}"/>
+    </joint>
+    <link name="front_beam">
+        <visual>
+            <geometry>
+                <box size="0.04 .34 .04" />
+            </geometry>
+            <origin rpy="0 0 0" xyz="0 0 0.025" />
+            <material name="black">
+                <color rgba="0 0 0 1" />
+            </material>
+        </visual>
+        <collision>
+            <origin xyz="0 0 .025"/>
+            <geometry>
+                <box size="0.04 0.34 0.04"/>
+            </geometry>
+        </collision>
+        <xacro:inertial_box mass="0.5" x="0.04" y="0.34" z="0.04">
+            <origin xyz="0 0 0" rpy="0 0 0"/>
+        </xacro:inertial_box>
+    </link>
+    <gazebo reference="front_beam">
+        <material>Gazebo/Black</material>
+    </gazebo>
     <joint name="base_to_second_layercylinder_1" type="fixed">
         <parent link="base_plate"/>

File: install/ayuda_description/share/ayuda_description/urdf/robotcar.urdf.xacro (robot description, xacro)
@@ -10,6 +10,6 @@
         <xacro:include filename="gazebo_control.xacro" />
     </xacro:unless>
-    <!-- <xacro:include filename="lidar.xacro" /> -->
-    <!-- <xacro:include filename="camera.xacro" /> -->
+    <xacro:include filename="lidar.xacro" />
+    <xacro:include filename="camera.xacro" />
     <!-- <xacro:include filename="depth_camera.xacro" /> -->
 </robot>

File: src/ayuda_description/urdf/camera.xacro (robot description, xacro)
@@ -2,5 +2,5 @@
 <robot xmlns:xacro="http://www.ros.org/wiki/xacro" >
     <joint name="camera_joint" type="fixed">
-        <parent link="chassis"/>
+        <parent link="base_plate"/>
         <child link="camera_link"/>
         <origin xyz="0.276 0 0.181" rpy="0 0.18 0"/>
@@ -32,5 +32,5 @@
             <pose> 0 0 0 0 0 0 </pose>
             <visualize>true</visualize>
-            <update_rate>10</update_rate>
+            <update_rate>30</update_rate>
             <camera>
                 <horizontal_fov>1.089</horizontal_fov>
